Commit message: Add transmission to right_vacuum_gripper.xacro

File: jsk_2016_01_baxter_apc/robots/right_vacuum_gripper.xacro (robot description, xacro)
@@ -209,3 +209,44 @@
     <limit lower="0" upper="3.14" effort="0" velocity="1.0"/>
   </joint>
+  <!--Transmission-->
+  <transmission name="right_gripper_prismatic_trans">
+    <type>transmission_interface/SimpleTransmission</type>
+    <joint name="right_gripper_prismatic_joint">
+      <hardwareInterface>PositionJointInterface</hardwareInterface>
+    </joint>
+    <actuator name="right_gripper_prismatic_joint_motor">
+      <hardwareInterface>PositionJointInterface</hardwareInterface>
+      <mechanicalReduction>0.024</mechanicalReduction>
+    </actuator>
+  </transmission>
+  <transmission name="right_gripper_vacuum_pad_trans">
+    <type>transmission_interface/SimpleTransmission</type>
+    <joint name="right_gripper_vacuum_pad_joint">
+      <hardwareInterface>PositionJointInterface</hardwareInterface>
+    </joint>
+    <actuator name="right_gripper_vacuum_pad_tendon_winder">
+      <hardwareInterface>PositionJointInterface</hardwareInterface>
+      <mechanicalReduction>1.46484375</mechanicalReduction>
+    </actuator>
+  </transmission>
+  <transmission name="right_gripper_finger_yaw_trans">
+    <type>transmission_interface/SimpleTransmission</type>
+    <joint name="right_gripper_finger_yaw_joint">
+      <hardwareInterface>PositionJointInterface</hardwareInterface>
+    </joint>
+    <actuator name="right_gripper_finger_yaw_joint_motor">
+      <hardwareInterface>PositionJointInterface</hardwareInterface>
+      <mechanicalReduction>1.5</mechanicalReduction>
+    </actuator>
+  </transmission>
+  <transmission name="right_gripper_finger_roll_trans">
+    <type>transmission_interface/SimpleTransmission</type>
+    <joint name="right_gripper_finger_roll_joint">
+      <hardwareInterface>PositionJointInterface</hardwareInterface>
+    </joint>
+    <actuator name="right_gripper_finger_tendon_winder">
+      <hardwareInterface>PositionJointInterface</hardwareInterface>
+      <mechanicalReduction>1.0</mechanicalReduction>
+    </actuator>
+  </transmission>
 </robot>

Commit message: Add right gripper-v5 collision

File: jsk_2016_01_baxter_apc/robots/right_vacuum_gripper.xacro (robot description, xacro)
@@ -19,7 +19,33 @@
   </gazebo>
   <!--Link bodies-->
+  <xacro:property name="base_rect_offset_x" value="0.0065" />
+  <xacro:property name="base_rect_l" value="0.2805" />
+  <xacro:property name="base_rect_h" value="0.107" />
+  <xacro:property name="base_rect_w" value="0.15" />
+  <xacro:property name="camera_rect_offset_x" value="-0.061" />
+  <xacro:property name="camera_rect_offset_y" value="-0.037" />
+  <xacro:property name="camera_rect_offset_z" value="0.004" />
+  <xacro:property name="camera_rect_l" value="0.04" />
+  <xacro:property name="camera_rect_h" value="0.03" />
+  <xacro:property name="camera_rect_w" value="0.165" />
+  <xacro:property name="tube_rect_offset_x" value="0.0475" />
+  <xacro:property name="tube_rect_offset_y" value="0.012" />
+  <xacro:property name="tube_rect_offset_z" value="0.17" />
+  <xacro:property name="tube_rect_l" value="0.29" />
+  <xacro:property name="tube_rect_h" value="0.034" />
+  <xacro:property name="tube_rect_w" value="0.081" />
   <xacro:property name="pad_with_base_offset_x" value="-0.048" />
   <xacro:property name="pad_with_base_offset_y" value="-0.0005" />
   <xacro:property name="pad_with_base_offset_z" value="-0.302" />
+  <xacro:property name="pad_with_base_col_z" value="0.0145" />
+  <xacro:property name="pad_with_base_rect_l" value="0.055" />
+  <xacro:property name="pad_with_base_rect_h" value="0.028" />
+  <xacro:property name="pad_with_base_rect_w" value="0.028" />
+  <xacro:property name="finger_base_rect_l" value="0.022" />
+  <xacro:property name="finger_base_rect_h" value="0.032" />
+  <xacro:property name="finger_base_rect_w" value="0.036" />
+  <xacro:property name="finger_rect_l" value="0.04" />
+  <xacro:property name="finger_rect_h" value="0.016" />
+  <xacro:property name="finger_rect_w" value="0.11" />
   <!--Joints-->
   <xacro:property name="hand_offset_x" value="-0.01" />
@@ -43,5 +69,16 @@
       </material>
     </visual>
-    <!--FIXME: Add collision-->
+    <collision>
+      <origin rpy="0 0 0" xyz="${base_rect_offset_x} 0 ${base_rect_l/2}"/>
+      <geometry>
+        <box size="${base_rect_h} ${base_rect_w} ${base_rect_l}"/>
+      </geometry>
+    </collision>
+    <collision>
+      <origin rpy="0 0 0" xyz="${camera_rect_offset_x} ${camera_rect_offset_y} ${camera_rect_offset_z}"/>
+      <geometry>
+        <box size="${camera_rect_h} ${camera_rect_w} ${camera_rect_l}"/>
+      </geometry>
+    </collision>
     <!--FIXME: Adjust inertia-->
     <inertial>
@@ -61,5 +98,10 @@
       </material>
     </visual>
-    <!--FIXME: Add collision-->
+    <collision>
+      <origin rpy="0 0 0" xyz="${tube_rect_offset_x} ${tube_rect_offset_y} ${tube_rect_offset_z}"/>
+      <geometry>
+        <box size="${tube_rect_h} ${tube_rect_w} ${tube_rect_l}"/>
+      </geometry>
+    </collision>
     <!--FIXME: Adjust inertia-->
     <inertial>
@@ -79,5 +121,10 @@
       </material>
     </visual>
-    <!--FIXME: Add collision-->
+    <collision>
+      <origin rpy="0 0 0" xyz="0 0 ${pad_with_base_col_z}"/>
+      <geometry>
+        <box size="${pad_with_base_rect_h} ${pad_with_base_rect_w} ${pad_with_base_rect_l}"/>
+      </geometry>
+    </collision>
     <!--FIXME: Adjust inertia-->
     <inertial>
@@ -97,5 +144,10 @@
       </material>
     </visual>
-    <!--FIXME: Add collision-->
+    <collision>
+      <origin rpy="0 0 0" xyz="0 0 ${-finger_base_rect_l/2}"/>
+      <geometry>
+        <box size="${finger_base_rect_h} ${finger_base_rect_w} ${finger_base_rect_l}"/>
+      </geometry>
+    </collision>
     <!--FIXME: Adjust inertia-->
     <inertial>
@@ -115,5 +167,10 @@
       </material>
     </visual>
-    <!--FIXME: Add collision-->
+    <collision>
+      <origin rpy="0 0 0" xyz="0 0 ${-finger_base_rect_l/2}"/>
+      <geometry>
+        <box size="${finger_base_rect_h} ${finger_base_rect_w} ${finger_base_rect_l}"/>
+      </geometry>
+    </collision>
     <!--FIXME: Adjust inertia-->
     <inertial>
@@ -133,5 +190,10 @@
       </material>
     </visual>
-    <!--FIXME: Add collision-->
+    <collision>
+      <origin rpy="0 0 0" xyz="0 ${-finger_rect_w/2} 0"/>
+      <geometry>
+        <box size="${finger_rect_h} ${finger_rect_w} ${finger_rect_l}"/>
+      </geometry>
+    </collision>
     <!--FIXME: Adjust inertia-->
     <inertial>
@@ -151,5 +213,10 @@
       </material>
     </visual>
-    <!--FIXME: Add collision-->
+    <collision>
+      <origin rpy="0 0 0" xyz="0 ${finger_rect_w/2} 0"/>
+      <geometry>
+        <box size="${finger_rect_h} ${finger_rect_w} ${finger_rect_l}"/>
+      </geometry>
+    </collision>
     <!--FIXME: Adjust inertia-->
     <inertial>

Commit message: Add calib_speed and increase joint speed

File: jsk_2016_01_baxter_apc/robots/right_vacuum_gripper.xacro (robot description, xacro)
@@ -237,5 +237,5 @@
     <child link="right_gripper_tube"/>
     <axis xyz="0 0 1"/>
-    <limit lower="0" upper="0.124" effort="0" velocity="0.024"/>
+    <limit lower="0" upper="0.124" effort="0" velocity="0.048"/>
   </joint>
   <joint name="right_gripper_vacuum_pad_joint" type="revolute">

Commit message: Maximize gripper joint speed

File: jsk_2016_01_baxter_apc/robots/right_vacuum_gripper.xacro (robot description, xacro)
@@ -244,5 +244,5 @@
     <child link="right_gripper_pad_with_base"/>
     <axis xyz="0 1 0"/>
-    <limit lower="-1.58" upper="1.58" effort="0" velocity="0.68"/>
+    <limit lower="-1.58" upper="1.58" effort="0" velocity="2.24"/>
   </joint>
   <joint name="right_gripper_finger_yaw_joint" type="revolute">
@@ -251,5 +251,5 @@
     <child link="right_gripper_l_finger_base"/>
     <axis xyz="0 0 1"/>
-    <limit lower="0" upper="1.58" effort="0" velocity="0.66"/>
+    <limit lower="0" upper="1.58" effort="0" velocity="0.76"/>
   </joint>
   <joint name="right_gripper_r_finger_yaw_joint" type="revolute">
@@ -259,5 +259,5 @@
     <mimic joint="right_gripper_finger_yaw_joint" multiplier="1"/>
     <axis xyz="0 0 -1"/>
-    <limit lower="0" upper="1.58" effort="0" velocity="0.66"/>
+    <limit lower="0" upper="1.58" effort="0" velocity="0.76"/>
   </joint>
   <joint name="right_gripper_finger_roll_joint" type="revolute">
@@ -266,5 +266,5 @@
     <child link="right_gripper_l_finger"/>
     <axis xyz="1 0 0"/>
-    <limit lower="0" upper="3.14" effort="0" velocity="1.0"/>
+    <limit lower="0" upper="3.14" effort="0" velocity="3.0"/>
   </joint>
   <joint name="right_gripper_r_finger_roll_joint" type="revolute">
@@ -274,5 +274,5 @@
     <mimic joint="right_gripper_finger_roll_joint" multiplier="1"/>
     <axis xyz="-1 0 0"/>
-    <limit lower="0" upper="3.14" effort="0" velocity="1.0"/>
+    <limit lower="0" upper="3.14" effort="0" velocity="3.0"/>
   </joint>
   <!--Transmission-->

Commit message: Refine rviz for demo

File: jsk_2016_01_baxter_apc/robots/right_vacuum_gripper.xacro (robot description, xacro)
@@ -108,6 +108,50 @@
         <mesh filename="package://jsk_2016_01_baxter_apc/meshes/visual/ideal_hand_stl/nozzle.stl" scale="0.001 0.001 0.001"/>
       </geometry>
-      <material name="black">
-        <color rgba="0 0 0 1"/>
+      <material name="green">
+        <color rgba="0 0.7 0 1"/>
+      </material>
+    </visual>
+  </link>
+  <link name="ver_cyl">
+    <visual>
+      <origin rpy="0 ${M_PI/2} 0" xyz="-0.040 0 0.040"/>
+      <geometry>
+        <cylinder radius="0.040" length="0.100"/>
+      </geometry>
+      <material name="blue">
+        <color rgba="0 0 1 1"/>
+      </material>
+    </visual>
+  </link>
+  <link name="box">
+    <visual>
+      <origin rpy="0 0 0" xyz="0.020 0 0.020"/>
+      <geometry>
+        <box size="0.100 0.080 0.040"/>
+      </geometry>
+      <material name="blue">
+        <color rgba="0 0 1 1"/>
+      </material>
+    </visual>
+  </link>
+  <link name="hor_cyl">
+    <visual>
+      <origin rpy="${M_PI/2} 0 0" xyz="-0.010 0 0.050"/>
+      <geometry>
+        <cylinder radius="0.030" length="0.100"/>
+      </geometry>
+      <material name="blue">
+        <color rgba="0 0 1 1"/>
+      </material>
+    </visual>
+  </link>
+  <link name="sphere">
+    <visual>
+      <origin rpy="0 0 0" xyz="0 0 0.035"/>
+      <geometry>
+        <sphere radius="0.035"/>
+      </geometry>
+      <material name="blue">
+        <color rgba="0 0 1 1"/>
       </material>
     </visual>
@@ -175,3 +219,23 @@
     <limit lower="-1.58" upper="1.58" effort="0" velocity="4.5"/>
   </joint>
+  <joint name="fixed_to_ver_cyl" type="fixed">
+    <origin rpy="0 0 0" xyz="0 0 0.030" />
+    <parent link="nozzle"/>
+    <child link="ver_cyl"/>
+  </joint>
+  <joint name="fixed_to_box" type="fixed">
+    <origin rpy="0 0 0" xyz="0 0 0.030" />
+    <parent link="nozzle"/>
+    <child link="box"/>
+  </joint>
+  <joint name="fixed_to_hor_cyl" type="fixed">
+    <origin rpy="0 0 0" xyz="0 0 0.180" />
+    <parent link="link0"/>
+    <child link="hor_cyl"/>
+  </joint>
+  <joint name="fixed_to_sphere" type="fixed">
+    <origin rpy="0 0 0" xyz="0 0 0.030" />
+    <parent link="nozzle"/>
+    <child link="sphere"/>
+  </joint>
 </robot>

Commit message: Fix urdf of gripper-v5

File: jsk_2016_01_baxter_apc/robots/right_vacuum_gripper.xacro (robot description, xacro)
@@ -63,8 +63,17 @@
       <origin rpy="${M_PI/2} 0 ${M_PI/2}" xyz="0 0 0"/>
       <geometry>
-        <mesh filename="package://jsk_2016_01_baxter_apc/meshes/visual/right_gripper_base.stl" scale="0.001 0.001 0.001"/>
-      </geometry>
-      <material name="lightgrey">
-        <color rgba="0.5 0.5 0.5 1"/>
+        <mesh filename="package://jsk_2016_01_baxter_apc/meshes/visual/right_gripper_base_main.stl" scale="0.001 0.001 0.001"/>
+      </geometry>
+      <material name="lightgrey">
+        <color rgba="0.5 0.5 0.5 1"/>
+      </material>
+    </visual>
+    <visual>
+      <origin rpy="${M_PI/2} 0 ${M_PI/2}" xyz="0 0 0"/>
+      <geometry>
+        <mesh filename="package://jsk_2016_01_baxter_apc/meshes/visual/right_gripper_palm_pad.stl" scale="0.001 0.001 0.001"/>
+      </geometry>
+      <material name="lightbrown">
+        <color rgba="0.6 0.5 0.2 1"/>
       </material>
     </visual>
@@ -92,8 +101,26 @@
       <origin rpy="${M_PI/2} 0 ${M_PI/2}" xyz="0 0 0"/>
       <geometry>
-        <mesh filename="package://jsk_2016_01_baxter_apc/meshes/visual/right_gripper_tube.stl" scale="0.001 0.001 0.001"/>
-      </geometry>
-      <material name="lightgrey">
-        <color rgba="0.5 0.5 0.5 1"/>
+        <mesh filename="package://jsk_2016_01_baxter_apc/meshes/visual/right_gripper_tube_connectors.stl" scale="0.001 0.001 0.001"/>
+      </geometry>
+      <material name="lightgrey">
+        <color rgba="0.5 0.5 0.5 1"/>
+      </material>
+    </visual>
+    <visual>
+      <origin rpy="${M_PI/2} 0 ${M_PI/2}" xyz="0 0 0"/>
+      <geometry>
+        <mesh filename="package://jsk_2016_01_baxter_apc/meshes/visual/right_gripper_tube_main.stl" scale="0.001 0.001 0.001"/>
+      </geometry>
+      <material name="white">
+        <color rgba="0.7 0.7 0.7 1"/>
+      </material>
+    </visual>
+    <visual>
+      <origin rpy="${M_PI/2} 0 ${M_PI/2}" xyz="0 0 0"/>
+      <geometry>
+        <mesh filename="package://jsk_2016_01_baxter_apc/meshes/visual/right_gripper_tube_gear.stl" scale="0.001 0.001 0.001"/>
+      </geometry>
+      <material name="blue">
+        <color rgba="0 0.24 0.82 1"/>
       </material>
     </visual>
@@ -115,8 +142,17 @@
       <origin rpy="${M_PI/2} 0 ${M_PI/2}" xyz="${pad_with_base_offset_x} ${pad_with_base_offset_y} ${pad_with_base_offset_z}"/>
       <geometry>
-        <mesh filename="package://jsk_2016_01_baxter_apc/meshes/visual/right_gripper_pad_with_base.stl" scale="0.001 0.001 0.001"/>
-      </geometry>
-      <material name="lightgrey">
-        <color rgba="0.5 0.5 0.5 1"/>
+        <mesh filename="package://jsk_2016_01_baxter_apc/meshes/visual/right_gripper_vacuum_pad_base.stl" scale="0.001 0.001 0.001"/>
+      </geometry>
+      <material name="lightgrey">
+        <color rgba="0.5 0.5 0.5 1"/>
+      </material>
+    </visual>
+    <visual>
+      <origin rpy="${M_PI/2} 0 ${M_PI/2}" xyz="${pad_with_base_offset_x} ${pad_with_base_offset_y} ${pad_with_base_offset_z}"/>
+      <geometry>
+        <mesh filename="package://jsk_2016_01_baxter_apc/meshes/visual/right_gripper_vacuum_pad.stl" scale="0.001 0.001 0.001"/>
+      </geometry>
+      <material name="green">
+        <color rgba="0 1 0 1"/>
       </material>
     </visual>
@@ -184,8 +220,17 @@
       <origin rpy="${M_PI/2} 0 ${M_PI}" xyz="0 0 0"/>
       <geometry>
-        <mesh filename="package://jsk_2016_01_baxter_apc/meshes/visual/finger.stl" scale="0.001 0.001 0.001"/>
-      </geometry>
-      <material name="lightgrey">
-        <color rgba="0.5 0.5 0.5 1"/>
+        <mesh filename="package://jsk_2016_01_baxter_apc/meshes/visual/finger_main.stl" scale="0.001 0.001 0.001"/>
+      </geometry>
+      <material name="lightgrey">
+        <color rgba="0.5 0.5 0.5 1"/>
+      </material>
+    </visual>
+    <visual>
+      <origin rpy="${M_PI/2} 0 ${M_PI}" xyz="0 0 0"/>
+      <geometry>
+        <mesh filename="package://jsk_2016_01_baxter_apc/meshes/visual/finger_pad.stl" scale="0.001 0.001 0.001"/>
+      </geometry>
+      <material name="lightbrown">
+        <color rgba="0.6 0.5 0.2 1"/>
       </material>
     </visual>
@@ -207,8 +252,17 @@
       <origin rpy="${M_PI/2} 0 0" xyz="0 0 0"/>
       <geometry>
-        <mesh filename="package://jsk_2016_01_baxter_apc/meshes/visual/finger.stl" scale="0.001 0.001 0.001"/>
-      </geometry>
-      <material name="lightgrey">
-        <color rgba="0.5 0.5 0.5 1"/>
+        <mesh filename="package://jsk_2016_01_baxter_apc/meshes/visual/finger_main.stl" scale="0.001 0.001 0.001"/>
+      </geometry>
+      <material name="lightgrey">
+        <color rgba="0.5 0.5 0.5 1"/>
+      </material>
+    </visual>
+    <visual>
+      <origin rpy="${M_PI/2} 0 0" xyz="0 0 0"/>
+      <geometry>
+        <mesh filename="package://jsk_2016_01_baxter_apc/meshes/visual/finger_pad.stl" scale="0.001 0.001 0.001"/>
+      </geometry>
+      <material name="lightbrown">
+        <color rgba="0.6 0.5 0.2 1"/>
       </material>
     </visual>
