Commit message: Add palm endpoint to baxterrgv5

File: jsk_2016_01_baxter_apc/robots/right_vacuum_gripper_v5.xacro (robot description, xacro)
@@ -58,4 +58,6 @@
   <xacro:property name="l_finger_base_offset_y" value="0.026" />
   <xacro:property name="r_finger_base_offset_y" value="-0.026" />
+  <xacro:property name="palm_offset_x" value="0.015" />
+  <xacro:property name="palm_offset_z" value="0.28" />
   <!--Link bodies-->
   <link name="right_gripper_base">
@@ -280,4 +282,5 @@
     </inertial>
   </link>
+  <link name="right_gripper_palm_endpoint"/>
   <!--Joints-->
   <joint name="right_gripper_base_fixed" type="fixed">
@@ -330,4 +333,9 @@
     <limit lower="0" upper="3.14" effort="0" velocity="3.0"/>
   </joint>
+  <joint name="right_gripper_palm_endpoint_fixed" type="fixed">
+    <origin rpy="0 ${M_PI} 0" xyz="${palm_offset_x} 0 ${palm_offset_z}" />
+    <parent link="right_gripper_base"/>
+    <child link="right_gripper_palm_endpoint"/>
+  </joint>
   <!--Transmission-->
   <transmission name="right_gripper_prismatic_trans">

Commit message: Increase speed and torque of gripper joints

File: jsk_2016_01_baxter_apc/robots/right_vacuum_gripper_v5.xacro (robot description, xacro)
@@ -294,5 +294,5 @@
     <child link="right_gripper_tube"/>
     <axis xyz="0 0 1"/>
-    <limit lower="0" upper="0.124" effort="0" velocity="0.048"/>
+    <limit lower="0" upper="0.124" effort="0" velocity="0.132"/>
   </joint>
   <joint name="right_gripper_vacuum_pad_joint" type="revolute">
@@ -301,5 +301,5 @@
     <child link="right_gripper_pad_with_base"/>
     <axis xyz="0 1 0"/>
-    <limit lower="-1.58" upper="1.58" effort="0" velocity="2.24"/>
+    <limit lower="-1.58" upper="1.58" effort="0" velocity="3.36"/>
   </joint>
   <joint name="right_gripper_finger_yaw_joint" type="revolute">
@@ -308,5 +308,5 @@
     <child link="right_gripper_l_finger_base"/>
     <axis xyz="0 0 1"/>
-    <limit lower="0" upper="1.58" effort="0" velocity="0.76"/>
+    <limit lower="0" upper="1.58" effort="0" velocity="4.23"/>
   </joint>
   <joint name="right_gripper_r_finger_yaw_joint" type="revolute">
@@ -316,5 +316,5 @@
     <mimic joint="right_gripper_finger_yaw_joint" multiplier="1"/>
     <axis xyz="0 0 -1"/>
-    <limit lower="0" upper="1.58" effort="0" velocity="0.76"/>
+    <limit lower="0" upper="1.58" effort="0" velocity="4.23"/>
   </joint>
   <joint name="right_gripper_finger_roll_joint" type="revolute">
@@ -323,5 +323,5 @@
     <child link="right_gripper_l_finger"/>
     <axis xyz="1 0 0"/>
-    <limit lower="0" upper="3.14" effort="0" velocity="3.0"/>
+    <limit lower="0" upper="3.14" effort="0" velocity="5.5"/>
   </joint>
   <joint name="right_gripper_r_finger_roll_joint" type="revolute">
@@ -331,5 +331,5 @@
     <mimic joint="right_gripper_finger_roll_joint" multiplier="1"/>
     <axis xyz="-1 0 0"/>
-    <limit lower="0" upper="3.14" effort="0" velocity="3.0"/>
+    <limit lower="0" upper="3.14" effort="0" velocity="5.5"/>
   </joint>
   <joint name="right_gripper_palm_endpoint_fixed" type="fixed">
