Commit message: Change kiva pod color

File: jsk_apc2015_common/models/kiva_pod/urdf/pod_lowres_convex.xacro (robot description, xacro)
@@ -12,5 +12,5 @@
       <origin rpy="0 0 0" xyz="0 0 0"/>
       <geometry><box size="${x_part_size}"/></geometry>
-      <material name="darkgray"><color rgba=".2 .2 .2 1"/></material>
+      <material name="darkgray"><color rgba="0 .4 1 1"/></material>
     </visual>
     <collision>
@@ -28,5 +28,5 @@
       <origin rpy="0 0 0" xyz="0 0 ${-z_size/2}"/>
       <geometry><box size="${z_part_size}"/></geometry>
-      <material name="darkgray"><color rgba=".2 .2 .2 1"/></material>
+      <material name="darkgray"><color rgba="0 .4 1 1"/></material>
     </visual>
     <collision>
@@ -43,5 +43,5 @@
       <origin rpy="0 0 0" xyz="0 0 -.22"/>
       <geometry><box size="${z_part_size}"/></geometry>
-      <material name="darkgray"><color rgba=".2 .2 .2 1"/></material>
+      <material name="darkgray"><color rgba="0 .4 1 1"/></material>
     </visual>
     <collision>
@@ -58,5 +58,5 @@
       <origin rpy="0 0 0" xyz="0 0 0"/>
       <geometry><box size="${z_part_size}"/></geometry>
-      <material name="darkgray"><color rgba=".2 .2 .2 1"/></material>
+      <material name="darkgray"><color rgba="0 .4 1 1"/></material>
     </visual>
     <collision>
@@ -73,5 +73,5 @@
       <origin rpy="0 0 0" xyz="0 0 .22"/>
       <geometry><box size="${z_part_size}"/></geometry>
-      <material name="darkgray"><color rgba=".2 .2 .2 1"/></material>
+      <material name="darkgray"><color rgba="0 .4 1 1"/></material>
     </visual>
     <collision>
@@ -88,5 +88,5 @@
       <origin rpy="0 0 0" xyz="0 0 ${z_size/2}"/>
       <geometry><box size="${z_part_size}"/></geometry>
-      <material name="darkgray"><color rgba=".2 .2 .2 1"/></material>
+      <material name="darkgray"><color rgba="0 .4 1 1"/></material>
     </visual>
     <collision>
@@ -104,5 +104,5 @@
       <origin rpy="0 0 0" xyz="0 ${y_size/2} 0"/>
       <geometry><box size="${y_part_size}"/></geometry>
-      <material name="darkgray"><color rgba=".2 .2 .2 1"/></material>
+      <material name="darkgray"><color rgba="0 .4 1 1"/></material>
     </visual>
     <collision>
@@ -119,5 +119,5 @@
       <origin rpy="0 0 0" xyz="0 0.16 0"/>
       <geometry><box size="${y_part_size}"/></geometry>
-      <material name="darkgray"><color rgba=".2 .2 .2 1"/></material>
+      <material name="darkgray"><color rgba="0 .4 1 1"/></material>
     </visual>
     <collision>
@@ -134,5 +134,5 @@
       <origin rpy="0 0 0" xyz="0 -.16 0"/>
       <geometry><box size="${y_part_size}"/></geometry>
-      <material name="darkgray"><color rgba=".2 .2 .2 1"/></material>
+      <material name="darkgray"><color rgba="0 .4 1 1"/></material>
     </visual>
     <collision>
@@ -149,5 +149,5 @@
       <origin rpy="0 0 0" xyz="0 -${y_size/2} 0"/>
       <geometry><box size="${y_part_size}"/></geometry>
-      <material name="darkgray"><color rgba=".2 .2 .2 1"/></material>
+      <material name="darkgray"><color rgba="0 .4 1 1"/></material>
     </visual>
     <collision>

Commit message: Change color from blue to red

File: jsk_apc2015_common/models/kiva_pod/urdf/pod_lowres_convex.xacro (robot description, xacro)
@@ -12,5 +12,5 @@
       <origin rpy="0 0 0" xyz="0 0 0"/>
       <geometry><box size="${x_part_size}"/></geometry>
-      <material name="darkgray"><color rgba="0 .4 1 1"/></material>
+      <material name="darkgray"><color rgba="1 0.3 0 1"/></material>
     </visual>
     <collision>
@@ -28,5 +28,5 @@
       <origin rpy="0 0 0" xyz="0 0 ${-z_size/2}"/>
       <geometry><box size="${z_part_size}"/></geometry>
-      <material name="darkgray"><color rgba="0 .4 1 1"/></material>
+      <material name="darkgray"><color rgba="1 0.3 0 1"/></material>
     </visual>
     <collision>
@@ -43,5 +43,5 @@
       <origin rpy="0 0 0" xyz="0 0 -.22"/>
       <geometry><box size="${z_part_size}"/></geometry>
-      <material name="darkgray"><color rgba="0 .4 1 1"/></material>
+      <material name="darkgray"><color rgba="1 0.3 0 1"/></material>
     </visual>
     <collision>
@@ -58,5 +58,5 @@
       <origin rpy="0 0 0" xyz="0 0 0"/>
       <geometry><box size="${z_part_size}"/></geometry>
-      <material name="darkgray"><color rgba="0 .4 1 1"/></material>
+      <material name="darkgray"><color rgba="1 0.3 0 1"/></material>
     </visual>
     <collision>
@@ -73,5 +73,5 @@
       <origin rpy="0 0 0" xyz="0 0 .22"/>
       <geometry><box size="${z_part_size}"/></geometry>
-      <material name="darkgray"><color rgba="0 .4 1 1"/></material>
+      <material name="darkgray"><color rgba="1 0.3 0 1"/></material>
     </visual>
     <collision>
@@ -88,5 +88,5 @@
       <origin rpy="0 0 0" xyz="0 0 ${z_size/2}"/>
       <geometry><box size="${z_part_size}"/></geometry>
-      <material name="darkgray"><color rgba="0 .4 1 1"/></material>
+      <material name="darkgray"><color rgba="1 0.3 0 1"/></material>
     </visual>
     <collision>
@@ -104,5 +104,5 @@
       <origin rpy="0 0 0" xyz="0 ${y_size/2} 0"/>
       <geometry><box size="${y_part_size}"/></geometry>
-      <material name="darkgray"><color rgba="0 .4 1 1"/></material>
+      <material name="darkgray"><color rgba="1 0.3 0 1"/></material>
     </visual>
     <collision>
@@ -119,5 +119,5 @@
       <origin rpy="0 0 0" xyz="0 0.16 0"/>
       <geometry><box size="${y_part_size}"/></geometry>
-      <material name="darkgray"><color rgba="0 .4 1 1"/></material>
+      <material name="darkgray"><color rgba="1 0.3 0 1"/></material>
     </visual>
     <collision>
@@ -134,5 +134,5 @@
       <origin rpy="0 0 0" xyz="0 -.16 0"/>
       <geometry><box size="${y_part_size}"/></geometry>
-      <material name="darkgray"><color rgba="0 .4 1 1"/></material>
+      <material name="darkgray"><color rgba="1 0.3 0 1"/></material>
     </visual>
     <collision>
@@ -149,5 +149,5 @@
       <origin rpy="0 0 0" xyz="0 -${y_size/2} 0"/>
       <geometry><box size="${y_part_size}"/></geometry>
-      <material name="darkgray"><color rgba="0 .4 1 1"/></material>
+      <material name="darkgray"><color rgba="1 0.3 0 1"/></material>
     </visual>
     <collision>
